File: eagle/sigma_mix.brd (EAGLE design)
At the start: 112 x 59.5 mm, 137 parts, among them J1 POWER_JACK, J2 RCA_JACK_CUI, J3 RCA_JACK_CUI, J4 RCA_JACK_CUI, J5 RCA_JACK_CUI, J6 RCA_JACK_X2_CUI, J7 RCA_JACK_X2_CUI, J8 RCA_JACK_X2_CUI, J9 RCA_JACK_X2_CUI, SW3 400MSP1R1BLKM7QE, SW4 OMRON_B3M, U3 ADM811TARTZ-REEL7, U4 ADAU1701JSTZ, U5 ADAU1701JSTZ, Y1 12.28MHz

Commit message: Update to v0.5.
Parts:
- removed C66, C68, C70, C71: 56nF, rcl:C2012
- removed JP7: (no value), pinhead:2X06
- removed R44, R45, R46, R47: 49k9, SparkFun:0603-RES
- removed U5: ADAU1701JSTZ, ADI-Phase-2:QFP50P900X900X160-48N
- added C30: 100uF, rcl:B/3528-21R
- added C4, C5: 0.1uF, rcl:C2012
- added C6: 10uF, rcl:R/2012-12R
- added LED1, LED2: (no value), myled:CHIPLED_1206
- added R28, R6: 8k06, SparkFun:0603-RES
- added R29, R5, R7: 56R2, SparkFun:0603-RES
- added R4: 10k, SparkFun:0603-RES
- added SV1: (no value), con-lstb:MA03-2
- added U1: (no value), tkrworks:SOIC8
- C1: value 0.1uF -> 1uF
- C10: value 100pF -> 10uF
- C11: value 100pF -> 10uF; device rcl:C2012 -> rcl:R/2012-12R
- C12: value 100pF -> 0.1uF
- C14, C16, C17, C46, C47, C51: value 10uF -> 0.1uF
- C15: device rcl:C2012 -> rcl:R/2012-12R
- C18: device rcl:R/2012-12R -> rcl:C2012
- C19, C3, C36: value 10uF -> 0.1uF; device rcl:R/2012-12R -> rcl:C2012
- C2: value 1uF -> 10uF; device rcl:C2012 -> rcl:R/2012-12R
- C20, C22, C26, C48, C52: value 0.1uF -> 10uF
- C23, C29, C39, C53: value 0.1uF -> 100uF; device rcl:C2012 -> rcl:B/3528-21R
- C24: value 10uF -> 56nF; device rcl:R/2012-12R -> rcl:C2012
- C25: value 10uF -> 3.3nF; device rcl:R/2012-12R -> rcl:C2012
- C27, C28: value 0.1uF -> 100pF
- C34: value 0.1uF -> 56nF
- C40: value 56nF -> 10uF
- C41: value 56nF -> 10uF; device rcl:C2012 -> rcl:R/2012-12R
- C42, C43: value 3.3nF -> 0.1uF
- C45: value 0.1uF -> 10uF; device rcl:C2012 -> rcl:R/2012-12R
- C54: value 10uF -> 56nF
- C55: value 10uF -> 3.3nF
- C56: value 100uF -> 10uF; device rcl:B/3528-21R -> rcl:C2012
- C57, C58: value 100uF -> 100pF; device rcl:B/3528-21R -> rcl:C2012
- C61, C62, C63: value 100uF -> 56nF; device rcl:B/3528-21R -> rcl:C2012
- C9: value 100pF -> 100uF; device rcl:C2012 -> rcl:B/3528-21R
- J2, J5: value RCA_JACK_CUI -> RCA_JACK_X2_CUI; device tkrworks:RCA_JACK_CUI -> tkrworks:RCA_JACK_X2_CUI
- J7, J8: value RCA_JACK_X2_CUI -> RCA_JACK_CUI; device tkrworks:RCA_JACK_X2_CUI -> tkrworks:RCA_JACK_CUI
- JP3: device con-lstb:MA03-2 -> pinhead:2X06
- R12: value 10k -> 18k
- R13: value 10k -> 475
- R14: value 10k -> 56R2
- R15, R16, R17: value 10k -> 49k9
- R18: value 8R06 -> 49k9
- R19, R20, R21: value 8R06 -> 10k
- R2: value 10k -> 562
- R23: value 10k -> 0
- R24: value 18k -> 1k
- R25: value 18k -> 56R2
- R26: value 1k -> 8k06
- R27: value 1k -> 56R2
- R3: value 0 -> 1k
- R30, R31: value 475 -> 49k9
- R32: value 56R2 -> 18k
- R33: value 56R2 -> 475
- R35, R36, R37, R38: value 56R2 -> 49k9
- R39: value 56R2 -> 10k
- R40, R41, R42: value 49k9 -> 10k
- R43: value 49k9 -> 562
- R8: value 49k9 -> 8k06
- R9: value 49k9 -> 56R2
- SW1, SW2: device special:EDG-04 -> special:EDG-02
- U2: value (none) -> ADM811TARTZ-REEL7; device tkrworks:SOIC8 -> ADI-Phase-2:SOT143P290X130-4N
- U3: value ADM811TARTZ-REEL7 -> ADAU1701JSTZ; device ADI-Phase-2:SOT143P290X130-4N -> ADI-Phase-2:QFP50P900X900X160-48N
- moved R9 63.3 mm to (38.7, 13.0), turned to 180 degrees
- moved J5 62.7 mm to (40.0, 3.90), turned to 180 degrees
- moved R30 60.1 mm to (93.9, 43.9), turned to 90 degrees
- moved J8 56.5 mm to (72.5, 57.5), turned to 90 degrees
- moved C63 55.6 mm to (102.2, 13.1), turned to 0 degrees
- moved J7 55.5 mm to (88.0, 57.4), turned to 90 degrees
- moved R38 55.5 mm to (94.1, 10.6)
- moved J2 53.6 mm to (58.8, 3.90), turned to 180 degrees
- moved C40 52.1 mm to (88.7, 43.9), turned to 90 degrees
- moved R13 51.6 mm to (38.7, 20.3), turned to 0 degrees
- moved R15 49.9 mm to (43.2, 10.7), turned to 0 degrees
- moved R41 49.9 mm to (88.4, 31.8), turned to 180 degrees
- moved C1 46.8 mm to (19.1, 13.9), turned to 270 degrees
- moved J4 46.5 mm to (41.5, 57.5)
- moved R39 43.9 mm to (88.4, 27.2), turned to 0 degrees
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- renumbered C65 to C31, C67 to C32, C69 to C33, JP4 to SV2, JP5 to X1, JP6 to X2, SW3 to S1, SW4 to S2, U6 to IC1
Connections:
- new net N$13: LED1.A, R2.1
- new net N$9: LED2.A, R43.1
- net *RESET: now also R4.2, U2.2, U3.5; no longer R2.2, U3.2, U5.5
- net ADC0_1: now also R8.2, U3.2; no longer R19.2, U4.2
- net ADC0_2: now also R28.2, U4.2; no longer R21.2, U5.2
- net ADC1_1: now also R6.2, U3.4; no longer R18.2, U4.4
- net ADC1_2: now also R26.2, U4.4; no longer R20.2, U5.4
- net ADDR0_1: now also R20.2, U3.7; no longer R12.2, U4.7
- net ADDR0_2: now also R40.2, U4.7; no longer R13.2, U5.7
- net ADDR1_1: now also R21.2, U3.20; no longer R14.2, U4.20
- net ADDR1_2: now also R41.2, U4.20; no longer R15.2, U5.20
- net BRD_RESET: now also U2.3; no longer U3.3
- net DVDD: now also C5.1, C6.+, C7.1, U3.13, U3.24; no longer C22.1, C24.+, C26.1, U4.13, U4.24
- net FLG: now also U1.4; no longer U2.4
- net GND: now also C11.-, C14.2, C15.-, C16.2, C17.2, C18.2, C19.2, C2.-, C3.2, C36.2, C4.2, C41.-, C42.2, C43.2, C45.-, C5.2, C57.2, C58.2, C6.-, C61.2, C62.2, C63.2, JP3.10, JP3.12, JP3.2, JP3.4, JP3.6, JP3.8, LED1.C, LED2.C, R18.1, R20.1, R21.1, R30.1, R31.1, R32.1, R35.1, R36.1, R37.1, R38.1, R4.1, U1.5, U1.6, U1.7, U1.8, U2.1, U3.12, U3.25, U3.30, U3.33, U3.37, U3.38, U3.42; no longer C10.2, C11.2, C18.-, C19.-, C2.2, C23.2, C24.-, C25.-, C26.2, C29.2, C3.-, C36.-, C39.2, C45.2, C53.2, C54.2, C55.2, C66.2, C68.2, C70.2, C71.2, C9.2, JP7.10, JP7.12, JP7.2, JP7.4, JP7.6, JP7.8, R13.1, R14.1, R2.1, R23.1, R24.1, R25.1, R43.1, R44.1, R45.1, R46.1, R47.1, R8.1, R9.1, U2.5, U2.6, U2.7, U2.8, U5.1, U5.12, U5.25, U5.30, U5.33, U5.37, U5.38, U5.42
- net MCLKI: now also R23.2, U3.32; no longer R3.2, U5.32
- net MP1_1: now also SV1.1, U3.10; no longer JP3.1, U4.10
- net MP1_2: now also U4.10; no longer U5.10
- net MP2_1: now also SV1.2, U3.29; no longer JP3.2, U4.29
- net MP2_2: now also U4.29; no longer U5.29
- net MP3_1: now also SV1.3, U3.28; no longer JP3.3, U4.28
- net MP3_2: now also U4.28; no longer U5.28
- net MP7_1: now also SV1.4, U3.14; no longer JP3.4, U4.14
- net MP7_2: now also U4.14; no longer U5.14
- net MP8_1: now also SV1.5, U3.27; no longer JP3.5, U4.27
- net MP8_2: now also U4.27; no longer U5.27
- net MP9_1: now also SV1.6, U3.26; no longer JP3.6, U4.26
- net MP9_2: now also U4.26; no longer U5.26
- net N$1: now also R3.1, U3.17; no longer R26.1, U4.17
- net N$10: now also C10.2, C27.1, R10.2; no longer C14.2, C9.1, R8.2
- net N$12: now also C10.1, R6.1; no longer C14.1, R18.1
- net N$15: now also C26.2, C28.1, R11.2; no longer C11.1, C15.2, R10.2
- net N$16: now also C26.1, R8.1; no longer C15.1, R19.1
- net N$19: now also C9.-, R5.1; no longer C60.-, R36.1
- net N$2: now also C24.2, R13.2; no longer C40.2, R30.2
- net N$20: now also J3.2; no longer J2.2
- net N$21: now also C23.-, R7.1; no longer C61.-, R37.1
- net N$22: now also C29.-, R9.1; no longer C62.-, R38.1
- net N$24: now also C30.-, R14.1; no longer C63.-, R39.1
- net N$26: now also J5.2, R14.2, R15.2; no longer J9.2, R39.2, R41.2
- net N$28: now also J5.3, R16.2, R9.2; no longer J9.3, R38.2, R43.2
- net N$3: now also C24.1, C25.1, U3.35; no longer C40.1, C42.1, U4.35
- net N$33: now also J2.2, R17.2, R7.2; no longer J8.2, R37.2, R45.2
- net N$34: now also C34.1, J2.3, R18.2, R5.2; no longer C71.1, J8.3, R36.2, R47.2
- net N$35: now also J4.2; no longer J3.2
- net N$36: now also R24.1, U4.17; no longer R27.1, U5.17
- net N$37: now also C36.1, C37.+, C38.1, U4.13, U4.24; no longer C23.1, C25.+, C27.1, U5.13, U5.24
- net N$38: now also C54.2, R33.2; no longer C41.2, R31.2
- net N$39: now also C54.1, C55.1, U4.35; no longer C41.1, C43.1, U5.35
- net N$4: now also C17.1, C18.1, U3.47; no longer C44.1, C46.1, U4.47
- net N$40: now also C48.1, U4.47; no longer C45.1, U5.47
- net N$41: now also C50.1, U4.41; no longer C51.1, U5.41
- net N$42: now also C51.1, C52.1, U4.40; no longer C53.1, C55.1, U5.40
- net N$44: now also R32.2, U4.3; no longer R25.2, U5.3
- net N$46: now also C40.2, C57.1, R30.2; no longer C10.1, C16.2, R9.2
- net N$47: now also C40.1, R26.1; no longer C16.1, R20.1
- net N$48: now also C56.2, C58.1, R31.2; no longer C12.1, C17.2, R11.2
- net N$49: now also C56.1, R28.1; no longer C17.1, R21.1
- net N$5: now also R23.1; no longer R3.1
- net N$50: now also C39.-, R25.1; no longer C56.-, R32.1
- net N$51: now also C53.-, R27.1; no longer C57.-, R33.1
- net N$52: now also C59.-, R29.1; no longer C58.-, R34.1
- net N$53: now also C60.-, R34.1; no longer C59.-, R35.1
- net N$54: now also C61.1, J9.2, R34.2; no longer C64.1, J7.2, R40.2
- net N$55: now also C62.1, J9.3, R29.2, R36.2; no longer C66.1, J7.3, R34.2, R42.2
- net N$56: now also C63.1, R27.2, R37.2; no longer C68.1, R33.2, R44.2
- net N$57: now also C64.1, R25.2, R38.2; no longer C70.1, R32.2, R46.2
- net N$58: now also J7.2; no longer J4.2
- net N$59: now also J8.2; no longer J5.2
- net N$6: now also C19.1, C20.1, U3.41; no longer C48.1, C50.1, U4.41
- net N$7: now also C21.1, C22.1, U3.40; no longer C52.1, C54.1, U4.40
- net N$8: now also R12.2, U3.3; no longer R24.2, U4.3
- net OUT_BCLK_1: now also U3.19, U4.9; no longer U4.19, U5.9
- net OUT_BCLK_2: now also U3.9, U4.19; no longer U4.9, U5.19
- net OUT_LRCLK_1: now also U3.16, U4.8; no longer U4.16, U5.8
- net OUT_LRCLK_2: now also U3.8, U4.16; no longer U4.8, U5.16
- net PA1: now also R2.2
- net PSW: now also U1.1; no longer U2.1
- net SCL: now also U3.23; no longer U5.23
- net SDA: now also U3.22; no longer U5.22
- net SELFBOOT_1: now also R22.2, U3.6; no longer R16.2, SW1.3, U4.6
- net SELFBOOT_2: now also R42.2, U4.6; no longer R17.2, SW2.3, U5.6
- net TDM_OUT_1: now also U3.15, U4.11; no longer U4.15, U5.11
- net TDM_OUT_2: now also U3.11, U4.15; no longer U4.11, U5.15
- net VDD: now also C11.+, C12.1, C14.1, C15.+, C16.1, C2.+, C25.2, C3.1, C4.1, C41.+, C42.1, C43.1, C44.1, C45.+, C46.1, C55.2, JP3.1, JP3.11, JP3.3, JP3.5, JP3.7, JP3.9, R13.1, R19.2, R24.2, R3.2, R33.1, R39.2, R43.2, SW1.3, SW1.4, SW2.3, SW2.4, U1.3, U2.4, U3.18, U3.34, U3.36, U3.39, U3.48; no longer C1.1, C18.+, C19.+, C20.1, C21.1, C28.1, C29.1, C3.+, C34.1, C36.+, C37.+, C38.1, C39.1, C42.2, C43.2, C7.1, JP7.1, JP7.11, JP7.3, JP7.5, JP7.7, JP7.9, R26.2, R27.2, R30.1, R31.1, SW1.5, SW1.6, SW1.7, SW1.8, SW2.5, SW2.6, SW2.7, SW2.8, U2.3, U3.4, U5.18, U5.34, U5.36, U5.39, U5.48
- net VIN: now also C1.1, U1.2; no longer C2.1, U2.2
- net VOUT0_1: now also C23.+, U3.46; no longer C61.+, U4.46
- net VOUT0_2: now also C53.+, U4.46; no longer C57.+, U5.46
- net VOUT1_1: now also C9.+, U3.45; no longer C60.+, U4.45
- net VOUT1_2: now also C39.+, U4.45; no longer C56.+, U5.45
- net VOUT2_1: now also C30.+, U3.44; no longer C63.+, U4.44
- net VOUT2_2: now also C60.+, U4.44; no longer C59.+, U5.44
- net VOUT3_1: now also C29.+, U3.43; no longer C62.+, U4.43
- net VOUT3_2: now also C59.+, U4.43; no longer C58.+, U5.43
- net WP_1: now also R19.1, U3.21; no longer R22.2, SW1.4, U4.21
- net WP_2: now also R39.1, U4.21; no longer R23.2, SW2.4, U5.21
Routing:
- net PA1: track 14.3 -> 46.1 mm
- net GND: track 136.1 -> 157.9 mm, vias 45 -> 43
- net SELFBOOT_2: track 9.10 -> 2.52 mm
- net SELFBOOT_1: track 9.32 -> 3.08 mm
- net MCLKI: track 40.3 -> 34.1 mm
- net VDD: track 100.4 -> 104.6 mm, vias 19 -> 22
- net WP_1: track 46.5 -> 42.5 mm
- net WP_2: track 28.8 -> 26.9 mm, vias 3 -> 4
- net N$9: track 0.00 -> 1.90 mm
- net N$13: track 0.00 -> 1.90 mm
- net ADC1_1: track 33.0 -> 31.4 mm
- net N$57: track 8.61 -> 7.41 mm
- net N$33: track 9.50 -> 8.30 mm
- net N$56: track 9.07 -> 7.87 mm
- net N$55: track 8.36 -> 7.16 mm
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Other:
- board text added: "1"
- board text added: "2"
- board text added: "3"
- board text added: "4"
- board text added: "L1"
- board text added: "L2"
- board text added: "R1"
- board text added: "R2"
- board text added: "for Turntablism & Portablism"
- board text added: "v0.5"
- board text removed: "SELF_BOOT"
- board text removed: "WP"
- board text removed: "v0.4"
